File: PCB/misterclippy.kicad_pcb (KiCad board)
At the start: 2 copper layers, 30.2 x 109.2 mm, 73 parts, among them J1 Audio In, J2 Audio In, J3 Through, J4 Through, J5 Input, J6 Input, J7 Output Gate, J8 Output Gate, J9 PWR, Q1 BC547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

Commit message: :art: Change transistor footprint for hand soldering
Parts:
- Q1, Q2: footprint Package_TO_SOT_THT:TO-92_Inline -> Package_TO_SOT_THT:TO-92_HandSolder
- moved Q2 0.23 mm to (111.0, 140.1)
- moved Q1 0.15 mm to (125.7, 140.1)
Routing:
- net Net-(Q1-C): track 12.9 -> 14.1 mm
- net Net-(Q1-B): track 13.6 -> 12.5 mm
- net Net-(Q2-B): track 12.3 -> 11.3 mm

Commit message: :wrench: Update resistor value in PCB
Parts:
- R14, R16: value 22k -> 15k
Changed lines of the file:
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@@
         (effects (font (size 1 1) (thickness 0.15)) (justify mirror))
     )
-    (fp_text value "22k" (at 3.81 -2.37) (layer "B.Fab")
+    (fp_text value "15k" (at 3.81 -2.37) (layer "B.Fab")
         (effects (font (size 1 1) (thickness 0.15)) (justify mirror))
     )
@@
         (effects (font (size 1 1) (thickness 0.15)) (justify mirror))
     )
-    (fp_text value "22k" (at 3.81 -2.37) (layer "B.Fab")
-        (effects (font (size 1 1) (thickness 0.15)) (justify mirror))
-    )
+    (fp_text value "15k" (at 3.81 -2.37) (layer "B.Fab")
+        (effects (font (size 1 1) (thickness 0.15)) (justify mirror))
+    )

Commit message: :wrench: Transfer new resistor values to PCB
Parts:
- R10, R11, R12, R4, R7, R9: value 100k -> 470k
- R13, R15: value 100k -> 22k
- R14, R16: value 15k -> 2k2
Changed lines of the file:
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@@
         (effects (font (size 1 1) (thickness 0.15)) (justify mirror))
     )
-    (fp_text value "100k" (at 3.81 -2.37) (layer "B.Fab")
+    (fp_text value "22k" (at 3.81 -2.37) (layer "B.Fab")
         (effects (font (size 1 1) (thickness 0.15)) (justify mirror))
     )
@@
         (effects (font (size 1 1) (thickness 0.15)) (justify mirror))
     )
-    (fp_text value "100k" (at 3.81 -2.37 90) (layer "B.Fab")
+    (fp_text value "470k" (at 3.81 -2.37 90) (layer "B.Fab")
         (effects (font (size 1 1) (thickness 0.15)) (justify mirror))
     )
@@
         (effects (font (size 1 1) (thickness 0.15)) (justify mirror))
     )
-    (fp_text value "100k" (at 3.81 -2.37 90) (layer "B.Fab")
+    (fp_text value "470k" (at 3.81 -2.37 90) (layer "B.Fab")
         (effects (font (size 1 1) (thickness 0.15)) (justify mirror))
     )
@@
         (effects (font (size 1 1) (thickness 0.15)) (justify mirror))
     )
-    (fp_text value "15k" (at 3.81 -2.37) (layer "B.Fab")
+    (fp_text value "2k2" (at 3.81 -2.37) (layer "B.Fab")
         (effects (font (size 1 1) (thickness 0.15)) (justify mirror))
     )
@@
         (effects (font (size 1 1) (thickness 0.15)) (justify mirror))
     )
-    (fp_text value "100k" (at 3.81 -2.37 90) (layer "B.Fab")
+    (fp_text value "470k" (at 3.81 -2.37 90) (layer "B.Fab")
         (effects (font (size 1 1) (thickness 0.15)) (justify mirror))
     )
@@
         (effects (font (size 1 1) (thickness 0.15)) (justify mirror))
     )
-    (fp_text value "100k" (at 3.81 -2.37 90) (layer "B.Fab")
+    (fp_text value "470k" (at 3.81 -2.37 90) (layer "B.Fab")
         (effects (font (size 1 1) (thickness 0.15)) (justify mirror))
     )
@@
         (effects (font (size 1 1) (thickness 0.15)) (justify mirror))
     )
-    (fp_text value "15k" (at 3.81 -2.37) (layer "B.Fab")
+    (fp_text value "2k2" (at 3.81 -2.37) (layer "B.Fab")
         (effects (font (size 1 1) (thickness 0.15)) (justify mirror))
     )
@@
         (effects (font (size 1 1) (thickness 0.15)) (justify mirror))
     )
-    (fp_text value "100k" (at 3.81 -2.37 90) (layer "B.Fab")
+    (fp_text value "470k" (at 3.81 -2.37 90) (layer "B.Fab")
         (effects (font (size 1 1) (thickness 0.15)) (justify mirror))
     )
@@
         (effects (font (size 1 1) (thickness 0.15)) (justify mirror))
     )
-    (fp_text value "100k" (at 3.81 -2.37 90) (layer "B.Fab")
+    (fp_text value "470k" (at 3.81 -2.37 90) (layer "B.Fab")
         (effects (font (size 1 1) (thickness 0.15)) (justify mirror))
     )
@@
         (effects (font (size 1 1) (thickness 0.15)) (justify mirror))
     )
-    (fp_text value "100k" (at 3.81 -2.37) (layer "B.Fab")
+    (fp_text value "22k" (at 3.81 -2.37) (layer "B.Fab")
         (effects (font (size 1 1) (thickness 0.15)) (justify mirror))
     )

Commit message: :pencil2: Fix name on CC label
Other:
- board text added: "CC-BY-SA 4.0 Patrick Pickel Stefan Haun"
- board text removed: "CC-BY-SA 4.0 Patrick Pichel Stefan Haun"
Changed lines of the file:
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@@
     (effects (font (size 0.6 0.6) (thickness 0.1) bold) (justify left bottom mirror))
   )
-  (gr_text "CC-BY-SA 4.0\nPatrick Pichel\nStefan Haun" (at 133.858 129.413 90) (layer "F.SilkS")
+  (gr_text "CC-BY-SA 4.0\nPatrick Pickel\nStefan Haun" (at 133.858 129.413 90) (layer "F.SilkS")
     (effects (font (size 0.6 0.6) (thickness 0.1) bold) (justify left bottom))
   )
